File: sensor_ble_geiger.kicad_pcb (KiCad board)
At the start: 2 copper layers, 111.3 x 49.4 mm, 45 parts, among them J1 Conn_01x02, J2 Geiger +, J3 Geiger -, J4 Conn_01x04, Q1 MMBTA42, Q2 MMBT3904, Q3 MMBT3904, Q4 BC847, U1 NE555D, U2 LT1308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

Commit message: Move to 3.3V
Parts:
- removed C2: 10uF, Resistor_THT:R_Axial_DIN0204_L3.6mm_D1.6mm_P5.08mm_Horizontal
- removed C3: 33nF, Resistor_SMD:R_0805_2012Metric
- removed C5: 100uF, Resistor_THT:R_Axial_DIN0204_L3.6mm_D1.6mm_P5.08mm_Horizontal
- removed D1: MBRS120, Diode_SMD:D_SMB
- removed L1: 4.7uH, Geiger:IND_SMD_CD43
- removed R1: 47k, Resistor_SMD:R_0805_2012Metric
- removed R4: 100k, Resistor_SMD:R_0805_2012Metric
- removed R7: 309K, Resistor_SMD:R_0805_2012Metric
- removed U1: NE555D, Package_SO:SOIC-8_3.9x4.9mm_P1.27mm
- removed U2: LT1308, Package_SO:SO-8_5.3x6.2mm_P1.27mm
- added IC1: ICM7555CD, Package_SO:SO-8_3.9x4.9mm_P1.27mm, F.Cu at (103.0, 39.4)
- moved C1 16.7 mm to (100.4, 34.6), turned to 90 degrees
- moved R6 14.0 mm to (104.9, 49.7)
- moved C10 11.1 mm to (113.0, 40.7)
- moved R5 8.75 mm to (109.3, 46.0), turned to -90 degrees
- moved Q1 8.61 mm to (109.2, 50.5)
- moved C4 8.14 mm to (93.5, 43.6)
- moved R3 7.63 mm to (97.2, 43.5), turned to 90 degrees
- moved L2 7.50 mm to (99.5, 51.2)
- moved J1 7.40 mm to (55.1, 63.2)
- moved Q2 6.57 mm to (105.5, 45.9), turned to 90 degrees
- moved R2 4.20 mm to (101.2, 44.3)
Connections:
- L2 pad 1: /VCC_5V -> /VCC_3.3V
- Q2 pad 3: Net-(C4-Pad1) -> Net-(Q2-Pad3)
- R2 pad 1: /VCC_5V -> /VCC_3.3V
Routing:
- net /18660_Input: track 90.8 -> 12.0 mm
- net /VCC_3.3V: track 100.3 -> 159.6 mm
- net /VCC_5V: track 48.1 -> 0.00 mm, vias 3 -> 0
- net Net-(D1-Pad2): track 21.2 -> 0.00 mm
- net Net-(Q2-Pad3): track 0.00 -> 11.9 mm
- net Net-(R5-Pad1): track 29.2 -> 18.9 mm, vias 2 -> 0
- net Net-(R1-Pad1): track 9.23 -> 0.00 mm
- net Net-(C4-Pad1): track 25.1 -> 16.5 mm, vias 2 -> 0
- net Net-(Q1-Pad2): track 14.8 -> 6.56 mm
- net Net-(R4-Pad1): track 5.92 -> 0.00 mm
- net Net-(C10-Pad2): track 18.2 -> 13.5 mm, vias 2 -> 0
- net Net-(R2-Pad2): track 13.1 -> 10.7 mm
- net Net-(C1-Pad1): track 4.42 -> 2.01 mm
- net Net-(C3-Pad1): track 2.17 -> 0.00 mm
